File: master/eagle/master-noavr.brd (EAGLE design)
At the start: 38 x 60 mm, 12 parts, among them IC2 FT232RL, IC3 L293D, T1 BC547, X1 PN61729-S

Commit message: Yes, we already fixed the ground plane!
Routing:
- net GND: track 17.7 -> 36.7 mm, vias 2 -> 5
- net VCC: track 105.9 -> 105.0 mm
Changed lines of the file:
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@@
 <layer number="27" name="tValues" color="7" fill="1" visible="yes" active="yes"/>
 <layer number="28" name="bValues" color="7" fill="1" visible="yes" active="yes"/>
-<layer number="29" name="tStop" color="7" fill="3" visible="yes" active="yes"/>
-<layer number="30" name="bStop" color="7" fill="6" visible="yes" active="yes"/>
-<layer number="31" name="tCream" color="7" fill="4" visible="yes" active="yes"/>
-<layer number="32" name="bCream" color="7" fill="5" visible="yes" active="yes"/>
-<layer number="33" name="tFinish" color="6" fill="3" visible="yes" active="yes"/>
-<layer number="34" name="bFinish" color="6" fill="6" visible="yes" active="yes"/>
-<layer number="35" name="tGlue" color="7" fill="4" visible="yes" active="yes"/>
-<layer number="36" name="bGlue" color="7" fill="5" visible="yes" active="yes"/>
-<layer number="37" name="tTest" color="7" fill="1" visible="yes" active="yes"/>
-<layer number="38" name="bTest" color="7" fill="1" visible="yes" active="yes"/>
-<layer number="39" name="tKeepout" color="4" fill="11" visible="yes" active="yes"/>
-<layer number="40" name="bKeepout" color="1" fill="11" visible="yes" active="yes"/>
-<layer number="41" name="tRestrict" color="4" fill="10" visible="yes" active="yes"/>
-<layer number="42" name="bRestrict" color="1" fill="10" visible="yes" active="yes"/>
-<layer number="43" name="vRestrict" color="2" fill="10" visible="yes" active="yes"/>
-<layer number="44" name="Drills" color="7" fill="1" visible="yes" active="yes"/>
-<layer number="45" name="Holes" color="7" fill="1" visible="yes" active="yes"/>
-<layer number="46" name="Milling" color="3" fill="1" visible="yes" active="yes"/>
-<layer number="47" name="Measures" color="7" fill="1" visible="yes" active="yes"/>
-<layer number="48" name="Document" color="7" fill="1" visible="yes" active="yes"/>
-<layer number="49" name="Reference" color="7" fill="1" visible="yes" active="yes"/>
+<layer number="29" name="tStop" color="7" fill="3" visible="no" active="yes"/>
+<layer number="30" name="bStop" color="7" fill="6" visible="no" active="yes"/>
+<layer number="31" name="tCream" color="7" fill="4" visible="no" active="yes"/>
+<layer number="32" name="bCream" color="7" fill="5" visible="no" active="yes"/>
+<layer number="33" name="tFinish" color="6" fill="3" visible="no" active="yes"/>
+<layer number="34" name="bFinish" color="6" fill="6" visible="no" active="yes"/>
+<layer number="35" name="tGlue" color="7" fill="4" visible="no" active="yes"/>
+<layer number="36" name="bGlue" color="7" fill="5" visible="no" active="yes"/>
+<layer number="37" name="tTest" color="7" fill="1" visible="no" active="yes"/>
+<layer number="38" name="bTest" color="7" fill="1" visible="no" active="yes"/>
+<layer number="39" name="tKeepout" color="4" fill="11" visible="no" active="yes"/>
+<layer number="40" name="bKeepout" color="1" fill="11" visible="no" active="yes"/>
+<layer number="41" name="tRestrict" color="4" fill="10" visible="no" active="yes"/>
+<layer number="42" name="bRestrict" color="1" fill="10" visible="no" active="yes"/>
+<layer number="43" name="vRestrict" color="2" fill="10" visible="no" active="yes"/>
+<layer number="44" name="Drills" color="7" fill="1" visible="no" active="yes"/>
+<layer number="45" name="Holes" color="7" fill="1" visible="no" active="yes"/>
+<layer number="46" name="Milling" color="3" fill="1" visible="no" active="yes"/>
+<layer number="47" name="Measures" color="7" fill="1" visible="no" active="yes"/>
+<layer number="48" name="Document" color="7" fill="1" visible="no" active="yes"/>
+<layer number="49" name="Reference" color="7" fill="1" visible="no" active="yes"/>
 <layer number="50" name="dxf" color="7" fill="1" visible="no" active="no"/>
 <layer number="51" name="tDocu" color="7" fill="1" visible="yes" active="yes"/>
@@
 <wire x1="18.235" y1="64.365" x2="16" y2="64.365" width="0.4064" layer="1"/>
 <wire x1="16" y1="64.365" x2="16" y2="64" width="0.4064" layer="1"/>
+<via x="11" y="39" extent="1-16" drill="1" shape="square"/>
+<wire x1="11" y1="39" x2="11" y2="46" width="0.4064" layer="16"/>
+<via x="11" y="46" extent="1-16" drill="1" shape="square"/>
+<via x="23" y="39" extent="1-16" drill="1" shape="square"/>
+<wire x1="23" y1="39" x2="11" y2="39" width="0.4064" layer="16"/>
 </signal>
 <signal name="N$4">
@@
 <wire x1="3.78" y1="35.05" x2="3.78" y2="27.43" width="0.4064" layer="1"/>
 <wire x1="3.78" y1="35.05" x2="3.78" y2="35.22" width="0.4064" layer="1"/>
-<wire x1="3.78" y1="35.22" x2="1" y2="38" width="0.4064" layer="1"/>
-<wire x1="1" y1="38" x2="1" y2="49" width="0.4064" layer="1"/>
-<wire x1="1" y1="49" x2="5" y2="53" width="0.4064" layer="1"/>
+<wire x1="3.78" y1="35.22" x2="2" y2="37" width="0.4064" layer="1"/>
+<wire x1="2" y1="37" x2="2" y2="50" width="0.4064" layer="1"/>
+<wire x1="2" y1="50" x2="5" y2="53" width="0.4064" layer="1"/>
 <wire x1="5" y1="53" x2="10" y2="53" width="0.4064" layer="1"/>
 <wire x1="10" y1="53" x2="13" y2="56" width="0.4064" layer="1"/>
